File: ram-fpga/ram-fpga.kicad_pcb (KiCad board)
At the start: 2 copper layers, 68 x 65 mm, 9 parts, among them J1 Conn_02x20_Odd_Even, U1 27128, U2 27128, U3 MC74LVXC3245, U4 MC74LVXC3245, U5 MC74LVXC3245, U6 MC74LVXC3245

Commit message: switch to smt header
Parts:
- J1: footprint Connector_IDC:IDC-Header_2x20_P2.54mm_Vertical -> Connector_PinHeader_2.54mm:PinHeader_2x20_P2.54mm_Vertical_SMD
- moved J1 24.1 mm to (161.7, 70.8)
Routing:
- net GND: track 36.5 -> 49.0 mm, vias 5 -> 6
- net /t/~r_trans_data: track 71.5 -> 65.2 mm
- net /a14_33: track 30.5 -> 34.5 mm
- net /a12_33: track 23.4 -> 27.1 mm
- net /t/~r_trans: track 124.9 -> 128.0 mm
- net /~ce_33: track 49.4 -> 46.3 mm
- net /a7_33: track 19.3 -> 22.4 mm
- net /~eo_33: track 61.0 -> 63.1 mm
- net /a6_33: track 13.5 -> 15.3 mm
- net +5V: track 120.9 -> 119.3 mm
- net /a10_33: track 55.2 -> 56.8 mm
- net +3V3: track 113.4 -> 114.8 mm
- net /a5_33: track 8.42 -> 9.77 mm
- net /d3_33: track 40.4 -> 41.5 mm
- net /a11_33: track 70.5 -> 71.6 mm
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Other:
- board size 68 x 65 mm -> 68 x 67 mm
